File: QuadLampDriver/QuadLampDriver.sch (KiCad schematic (older format))
At the start: 2 parts

Commit message: Add the first few components (voltage divider)
Parts:
- added R?: 47k, symbol Device:R
- added R?: 10k, symbol Device:R
Connections:
- new net: R?.1, R?.2
- new net Control: R?.1
- new net GND: R?.2
Changed lines of the file:
@@
 EESchema Schematic File Version 4
+LIBS:QuadLampDriver-cache
 EELAYER 26 0
 EELAYER END
@@
 	1    0    0    -1
 $EndComp
+$Comp
+L Device:R R?
+U 1 1 5F286175
+P 1600 1350
+F 0 "R?" H 1670 1396 50  0000 L CNN
+F 1 "47k" H 1670 1305 50  0000 L CNN
+F 2 "" V 1530 1350 50  0001 C CNN
+F 3 "~" H 1600 1350 50  0001 C CNN
+	1    1600 1350
+	1    0    0    -1
+$EndComp
+$Comp
+L Device:R R?
+U 1 1 5F286233
+P 1600 1950
+F 0 "R?" H 1670 1996 50  0000 L CNN
+F 1 "10k" H 1670 1905 50  0000 L CNN
+F 2 "" V 1530 1950 50  0001 C CNN
+F 3 "~" H 1600 1950 50  0001 C CNN
+	1    1600 1950
+	1    0    0    -1
+$EndComp
+Wire Wire Line
+	1600 1500 1600 1800
+$Comp
+L power:GND #PWR?
+U 1 1 5F28A2F6
+P 1600 2100
+F 0 "#PWR?" H 1600 1850 50  0001 C CNN
+F 1 "GND" H 1605 1927 50  0000 C CNN
+F 2 "" H 1600 2100 50  0001 C CNN
+F 3 "" H 1600 2100 50  0001 C CNN
+	1    1600 2100
+	1    0    0    -1
+$EndComp
+Text GLabel 1400 1050 0    50   Input ~ 0
+Control
+Wire Wire Line
+	1600 1050 1400 1050
+Wire Wire Line
+	1600 1200 1600 1050
 $EndSCHEMATC

Commit message: Add inputs and outputs, and replicate circuit
Parts:
- added R? (x3): 47k, symbol Device:R
- added R? (x3): 10k, symbol Device:R
- added U? (x4): VN7007AHTR, symbol vn7007ahtr:VN7007AHTR
Connections:
- net labels added: +12V, ControlA, ControlB, ControlC, ControlD, OutputA, OutputB, OutputC, OutputD
- net labels removed: Control
- wire segments 3 -> 76

Commit message: Adjustments to lamp SSR boards
Parts:
- added R11, R16, R3, R7: 1k, symbol Device:R
- added R12, R4, R8, R?: 15k, symbol Device:R
- R1, R10, R13, R14, R2, R5, R6, R9: renamed from R?; footprint (none) -> Resistor_THT:R_Axial_DIN0309_L9.0mm_D3.2mm_P12.70mm_Horizontal
- gave numbers to parts that had none: 6
Connections:
- wire segments 76 -> 104

Commit message: Add low-power drivers for sidelight and indicator, and add output connector
Parts:
- added C? (x6): C, symbol Device:C
- added J?: Conn_01x06, symbol Connector_Generic:Conn_01x06
- added Q? (x2): FDC6330L, Package_TO_SOT_SMD:TSOT-23-6, symbol Transistor_FET:FDC6330L
- added R? (x8): R, symbol Device:R
Connections:
- wire segments 104 -> 189
